Commit message: implemented camera as macro for multiple placement

File: ros2_ws/src/simulation/urdf/camera.xacro (robot description, xacro)
@@ -1,68 +1,66 @@
 <?xml version="1.0"?>
 <robot xmlns:xacro="http://www.ros.org/wiki/xacro">
-    <joint name="camera_right_joint" type="fixed">
-        <parent link="base_link" />
-        <child link="camera_right_link" />
-        <origin xyz="2 0 1"
-            rpy="0 0 3.14" />
-    </joint>
-    <link name="camera_right_link">
-        <visual>
-            <geometry>
-                <box size="0.03 0.03 0.03" />
-            </geometry>
-            <material name="black" />
-        </visual>
-    </link>
-    <joint name="camera_right_optical_joint" type="fixed">
-        <parent link="camera_right_link" />
-        <child link="camera_right_link_optical" />
-        <origin xyz="0 0 0" rpy="0 0 0" />
-    </joint>
-    <link name="camera_right_link_optical"></link>
-    <gazebo reference="camera_right_link">
-        <material>Gazebo/Black</material>
-        <sensor name="wideangle_camera" type="wideanglecamera">
-            <camera>
-                <horizontal_fov>3.14</horizontal_fov>
-                <image>
-                    <width>800</width>
-                    <height>600</height>
-                </image>
-                <clip>
-                    <near>0.1</near>
-                    <far>100</far>
-                </clip>
-                <!-- A new section named `lens`. -->
-                <lens>
-                    <!-- type element is mandatory -->
-                    <type>custom</type>
-                    <!-- manually defined mapping function r = c1*f*fun(theta/c2 + c3) -->
-                    <!-- More information here:
+    <xacro:macro name="camera_macro" params="name parent_link x y z roll pitch yaw">
+        <joint name="${name}_joint" type="fixed">
+            <parent link="${parent_link}" />
+            <child link="${name}_link" />
+            <origin xyz="${x} ${y} ${z}" rpy="${roll} ${pitch} ${yaw}" />
+        </joint>
+        <link name="${name}_link">
+            <visual>
+                <geometry>
+                    <box size="0.1 0.1 0.1" /> <!-- Example camera size -->
+                </geometry>
+                <material name="black" />
+            </visual>
+        </link>
+        <gazebo reference="${name}_link">
+            <material>Gazebo/Black</material>
+            <sensor name="${name}" type="wideanglecamera">
+                <camera>
+                    <horizontal_fov>3.14</horizontal_fov>
+                    <image>
+                        <width>800</width>
+                        <height>600</height>
+                    </image>
+                    <clip>
+                        <near>0.1</near>
+                        <far>100</far>
+                    </clip>
+                    <!-- A new section named `lens`. -->
+                    <lens>
+                        <!-- type element is mandatory -->
+                        <type>custom</type>
+                        <!-- manually defined mapping function r = c1*f*fun(theta/c2 + c3) -->
+                        <!-- More information here:
                     https://en.wikipedia.org/wiki/Fisheye_lens#Mapping_function -->
-                    <custom_function>
-                        <c1>1.05</c1>
-                        <!-- linear scaling -->
-                        <c2>4</c2>
-                        <!-- angle scaling -->
-                        <f>1.0</f>
-                        <!-- one more scaling parameter -->
-                        <fun>tan</fun>
-                        <!-- one of sin,tan,id -->
-                    </custom_function>
-                    <!-- if it is set to `true` your horizontal FOV will ramain as defined -->
-                    <!-- othervise it depends on lens type and custom function, if there is one -->
-                    <scale_to_hfov>true</scale_to_hfov>
-                    <!-- clip everything that is outside of this angle -->
-                    <cutoff_angle>3.1415</cutoff_angle>
-                    <!-- resolution of the cubemap texture, the highter it is - the sharper is your
+                        <custom_function>
+                            <c1>1.05</c1>
+                            <!-- linear scaling -->
+                            <c2>4</c2>
+                            <!-- angle scaling -->
+                            <f>1.0</f>
+                            <!-- one more scaling parameter -->
+                            <fun>tan</fun>
+                            <!-- one of sin,tan,id -->
+                        </custom_function>
+                        <!-- if it is set to `true` your horizontal FOV will ramain as defined -->
+                        <!-- othervise it depends on lens type and custom function, if there is
+                            one -->
+                        <scale_to_hfov>true</scale_to_hfov>
+                        <!-- clip everything that is outside of this angle -->
+                        <cutoff_angle>3.1415</cutoff_angle>
+                        <!-- resolution of the cubemap texture, the highter it is - the sharper
+                            is
+                        your
                     image -->
-                    <env_texture_size>512</env_texture_size>
-                </lens>
-            </camera>
-            <always_on>1</always_on>
-            <update_rate>30</update_rate>
-            <topic>wide_angle_camera</topic>
-        </sensor>
-    </gazebo>
+                        <env_texture_size>512</env_texture_size>
+                    </lens>
+                </camera>
+                <always_on>1</always_on>
+                <update_rate>30</update_rate>
+                <topic>/camera/${name}</topic>
+            </sensor>
+        </gazebo>
+    </xacro:macro>
 </robot>

File: ros2_ws/src/simulation/urdf/robot.urdf.xacro (robot description, xacro)
@@ -15,10 +15,4 @@
     <!-- Base Link -->
     <link name="base_link">
-        <collision>
-            <origin xyz="0 0 1" rpy="0 0 0" />
-            <geometry>
-                <box size="1 1 1" />
-            </geometry>
-        </collision>
         <visual>
             <origin xyz="0 0 1" rpy="0 0 0" />
@@ -28,13 +22,22 @@
             <material name="orange" />
         </visual>
+        <visual>
+            <origin rpy="0 0 0" xyz="0 0 1" />
+            <geometry>
+                <box size="1 1 1" />
+            </geometry>
+            <material name="orange" />
+        </visual>
         <inertial>
-            <origin xyz="0 0 1" rpy="0 0 0" />
+            <origin rpy="0 0 0" xyz="0 0 1" />
             <mass value="1" />
-            <inertia
-                ixx="0.01" ixy="0.0" ixz="0.0"
-                iyy="0.01" iyz="0.0"
-                izz="0.01" />
+            <inertia ixx="0.01" ixy="0.0" ixz="0.0" iyy="0.01" iyz="0.0" izz="0.01" />
         </inertial>
     </link>
     <xacro:include filename="camera.xacro" />
+    <xacro:camera_macro name="top_view_camera_front" parent_link="base_link" x="-1.0" y="0.0"
+        z="0.3"
+        roll="0.0" pitch="0.0" yaw="0.0" />
+    <xacro:camera_macro name="top_view_camera_rear" parent_link="base_link" x="1.0" y="0.0" z="0.3"
+        roll="0.0" pitch="0.0" yaw="3.14" />
 </robot>

Commit message: made generic world creation from xacro and camera and lidar completely generic from xacro and integrated ros gz bridge with rviz

File: ros2_ws/src/simulation/urdf/camera.xacro (robot description, xacro)
@@ -1,4 +1,5 @@
 <?xml version="1.0"?>
 <robot xmlns:xacro="http://www.ros.org/wiki/xacro">
+    <xacro:include filename="$(find simulation)/worlds/utils.xacro" />
     <xacro:macro name="camera_macro" params="name parent_link x y z roll pitch yaw">
         <joint name="${name}_joint" type="fixed">
@@ -8,9 +9,8 @@
         </joint>
         <link name="${name}_link">
-            <visual>
+            <visual name="${name}_visual">
                 <geometry>
                     <box size="0.1 0.1 0.1" /> <!-- Example camera size -->
                 </geometry>
-                <material name="black" />
             </visual>
         </link>
@@ -48,5 +48,5 @@
                         <!-- othervise it depends on lens type and custom function, if there is
                             one -->
-                        <scale_to_hfov>true</scale_to_hfov>
+                        <scale_to_hfov>false</scale_to_hfov>
                         <!-- clip everything that is outside of this angle -->
                         <cutoff_angle>3.1415</cutoff_angle>
@@ -60,5 +60,8 @@
                 <always_on>1</always_on>
                 <update_rate>30</update_rate>
-                <topic>/camera/${name}</topic>
+                <topic>/camera/${name}/image</topic>
+                <camera_info>
+                    <topic>/camera/${name}/camera_info</topic>
+                </camera_info>
             </sensor>
         </gazebo>

File: ros2_ws/src/simulation/urdf/robot.urdf.xacro (robot description, xacro)
@@ -1,34 +1,22 @@
 <?xml version="1.0"?>
-<robot name="my_robot" xmlns:xacro="http://www.ros.org/wiki/xacro">
-    <!-- Define properties for reuse -->
-    <xacro:property name="lidar_range" value="10.0" />
-    <xacro:property name="lidar_resolution" value="0.01" />
-    <xacro:property name="camera_width" value="640" />
-    <xacro:property name="camera_height" value="480" />
-    <xacro:property name="camera_fov" value="1.57" />
-    <link name="world"></link>
+<robot name="vehicle" xmlns:xacro="http://www.ros.org/wiki/xacro">
+    <xacro:include filename="$(find simulation)/worlds/utils.xacro" />
+    <link name="world_link"></link>
     <joint name="base_joint" type="fixed">
         <origin xyz="0 0 0" rpy="0 0 0" />
         <parent link="world" />
         <child link="base_link" />
+        <origin xyz="0 0 0.0" rpy="0 0 0" />
     </joint>
     <!-- Base Link -->
     <link name="base_link">
-        <visual>
-            <origin xyz="0 0 1" rpy="0 0 0" />
+        <visual name="base_link_visual">
+            <origin xyz="0 0 0.25" rpy="0 0 0" />
             <geometry>
-                <box size="1 1 1" />
+                <box size="0.5 0.5 0.5" />
             </geometry>
-            <material name="orange" />
-        </visual>
-        <visual>
-            <origin rpy="0 0 0" xyz="0 0 1" />
-            <geometry>
-                <box size="1 1 1" />
-            </geometry>
-            <material name="orange" />
         </visual>
         <inertial>
-            <origin rpy="0 0 0" xyz="0 0 1" />
+            <origin rpy="0 0 0" xyz="0 0 0" />
             <mass value="1" />
             <inertia ixx="0.01" ixy="0.0" ixz="0.0" iyy="0.01" iyz="0.0" izz="0.01" />
@@ -36,8 +24,9 @@
     </link>
     <xacro:include filename="camera.xacro" />
-    <xacro:camera_macro name="top_view_camera_front" parent_link="base_link" x="-1.0" y="0.0"
-        z="0.3"
-        roll="0.0" pitch="0.0" yaw="0.0" />
-    <xacro:camera_macro name="top_view_camera_rear" parent_link="base_link" x="1.0" y="0.0" z="0.3"
-        roll="0.0" pitch="0.0" yaw="3.14" />
+    <xacro:camera_macro name="top_view_camera_front" parent_link="base_link" x="1.0" y="0.0" z="0.3" roll="0.0" pitch="0.0" yaw="0.0" />
+    <xacro:camera_macro name="top_view_camera_left" parent_link="base_link" x="0.0" y="0.5" z="0.3" roll="0.0" pitch="0.0" yaw="1.5" />
+    <xacro:camera_macro name="top_view_camera_right" parent_link="base_link" x="0.0" y="-0.5" z="0.3" roll="0.0" pitch="0.0" yaw="-1.5" />
+    <xacro:camera_macro name="top_view_camera_rear" parent_link="base_link" x="-1.0" y="0.0" z="0.3" roll="0.0" pitch="0.0" yaw="3.14" />
+    <xacro:include filename="lidar.xacro" />
+    <xacro:lidar_macro name="ref_lidar" parent_link="base_link" x="0.0" y="0.0" z="1.0" roll="0.0" pitch="0.0" yaw="0.0" />
 </robot>
