Commit message: made lidar appear in rviz and integrated gpu

File: ros2_ws/src/simulation/urdf/lidar.xacro (robot description, xacro)
@@ -22,4 +22,5 @@
                 <pose relative_to="${name}_link">0 0 0 0 0 0</pose>
                 <topic>/lidar/${name}</topic>
+                <gz_frame_id>${name}_link</gz_frame_id>
                 <update_rate>10</update_rate>
                 <ray>
@@ -27,13 +28,13 @@
                         <horizontal>
                             <samples>640</samples>
-                            <resolution>1</resolution>
-                            <min_angle>-1.396263</min_angle>
-                            <max_angle>1.396263</max_angle>
+                            <resolution>0.01</resolution>
+                            <min_angle>-3.14</min_angle>
+                            <max_angle>3.14</max_angle>
                         </horizontal>
                         <vertical>
-                            <samples>1</samples>
+                            <samples>50</samples>
                             <resolution>0.01</resolution>
-                            <min_angle>0</min_angle>
-                            <max_angle>0</max_angle>
+                            <min_angle>-0.5</min_angle>
+                            <max_angle>0.5</max_angle>
                         </vertical>
                     </scan>
@@ -41,9 +42,9 @@
                         <min>0.08</min>
                         <max>10.0</max>
-                        <resolution>0.01</resolution>
+                        <resolution>0.001</resolution>
                     </range>
                 </ray>
                 <always_on>1</always_on>
-                <visualize>true</visualize>
+                <visualize>false</visualize>
             </sensor>
         </gazebo>

File: ros2_ws/src/simulation/worlds/generic.urdf.xacro (robot description, xacro)
@@ -99,5 +99,4 @@
 			<direction>-0.5 0.1 -0.9</direction>
 		</light>
-		<link name="world_link"></link>
 		<model name="ground_plane">
 			<static>true</static>
