Commit message: switched world_link to world

File: ros2_ws/src/simulation/urdf/robot.urdf.xacro (robot description, xacro)
@@ -2,5 +2,5 @@
 <robot name="vehicle" xmlns:xacro="http://www.ros.org/wiki/xacro">
     <xacro:include filename="$(find simulation)/worlds/utils.xacro" />
-    <link name="world_link"></link>
+    <link name="world"></link>
     <joint name="base_joint" type="fixed">
         <origin xyz="0 0 0" rpy="0 0 0" />
