Commit message: implemented pinhole camera with bbox and integrated all 5 Lidars on rough positions with automated first module with groundtruth markers

File: ros2_ws/src/simulation/urdf/camera_wideangle.xacro (robot description, xacro)
@@ -2,5 +2,5 @@
 <robot xmlns:xacro="http://www.ros.org/wiki/xacro">
     <xacro:include filename="$(find simulation)/worlds/utils.xacro" />
-    <xacro:macro name="camera_macro" params="name parent_link x y z roll pitch yaw">
+    <xacro:macro name="camera_wideangle_macro" params="name parent_link x y z roll pitch yaw">
         <joint name="${name}_joint" type="fixed">
             <parent link="${parent_link}" />

File: ros2_ws/src/simulation/urdf/lidar.xacro (robot description, xacro)
@@ -6,5 +6,5 @@
             <parent link="${parent_link}" />
             <child link="${name}_link" />
-            <origin xyz="${x} ${y} ${z}" rpy="${roll} ${pitch} ${yaw}" />
+            <origin xyz="${x} ${y} ${z}" rpy="${roll * pi / 180.0} ${pitch * pi / 180.0} ${yaw * pi / 180.0}" />
         </joint>
         <link name="${name}_link">
@@ -42,5 +42,5 @@
                         <min>0.08</min>
                         <max>10.0</max>
-                        <resolution>0.001</resolution>
+                        <resolution>0.0001</resolution>
                     </range>
                 </ray>

File: ros2_ws/src/simulation/urdf/robot.urdf.xacro (robot description, xacro)
@@ -23,10 +23,30 @@
         </inertial>
     </link>
-    <xacro:include filename="camera.xacro" />
-    <xacro:camera_macro name="top_view_camera_front" parent_link="base_link" x="1.0" y="0.0" z="0.3" roll="0.0" pitch="0.0" yaw="0.0" />
-    <xacro:camera_macro name="top_view_camera_left" parent_link="base_link" x="0.0" y="0.5" z="0.3" roll="0.0" pitch="0.0" yaw="1.5" />
-    <xacro:camera_macro name="top_view_camera_right" parent_link="base_link" x="0.0" y="-0.5" z="0.3" roll="0.0" pitch="0.0" yaw="-1.5" />
-    <xacro:camera_macro name="top_view_camera_rear" parent_link="base_link" x="-1.0" y="0.0" z="0.3" roll="0.0" pitch="0.0" yaw="3.14" />
+    <xacro:include filename="camera_pinhole_bbox.xacro" />
+    <xacro:camera_pinhole_macro name="top_view_camera_front" parent_link="base_link"
+        hfov="140.0" width="640" height="480"
+        x="1.0" y="0.0" z="0.3"
+        roll="0.0" pitch="0.0" yaw="0.0"
+    />
+    <xacro:camera_pinhole_macro name="top_view_camera_left" parent_link="base_link"
+        hfov="140.0" width="640" height="480"
+        x="0.0" y="0.5" z="0.3"
+        roll="0.0" pitch="0.0" yaw="90"
+    />
+    <xacro:camera_pinhole_macro name="top_view_camera_right" parent_link="base_link"
+        hfov="140.0" width="640" height="480"
+        x="0.0" y="-0.5" z="0.3"
+        roll="0.0" pitch="0.0" yaw="-90"
+    />
+    <xacro:camera_pinhole_macro name="top_view_camera_rear" parent_link="base_link"
+        hfov="140.0" width="640" height="480"
+        x="-1.0" y="0.0" z="0.3"
+        roll="0.0" pitch="0.0" yaw="180"
+    />
     <xacro:include filename="lidar.xacro" />
-    <xacro:lidar_macro name="ref_lidar" parent_link="base_link" x="0.0" y="0.0" z="1.0" roll="0.0" pitch="0.0" yaw="0.0" />
+    <xacro:lidar_macro name="ref_lidar" parent_link="base_link" x="0.0" y="0.0" z="1.5" roll="0.0" pitch="0.0" yaw="0.0" />
+    <xacro:lidar_macro name="ref_lidar_front" parent_link="base_link" x="1.0" y="0.0" z="0.8" roll="0.0" pitch="25.0" yaw="0.0" />
+    <xacro:lidar_macro name="ref_lidar_right" parent_link="base_link" x="0.0" y="-0.5" z="0.8" roll="0.0" pitch="25.0" yaw="-90" />
+    <xacro:lidar_macro name="ref_lidar_rear" parent_link="base_link" x="-1.0" y="0.0" z="0.8" roll="0.0" pitch="25.0" yaw="180" />
+    <xacro:lidar_macro name="ref_lidar_left" parent_link="base_link" x="0.0" y="0.5" z="0.8" roll="0.0" pitch="25.0" yaw="90" />
 </robot>

File: ros2_ws/src/simulation/worlds/generic.urdf.xacro (robot description, xacro)
@@ -14,5 +14,4 @@
 			filename="gz-sim-sensors-system"
 			name="gz::sim::systems::Sensors">
-			<render_engine>ogre2</render_engine>
 		</plugin>
 		<plugin
@@ -125,9 +124,12 @@
 			</link>
 		</model>
-		<xacro:module_macro name="module_01" parent_link="world" x="5.0" y="0.0" z="0.0" roll="0.0" pitch="0.0" yaw="0.0" />
-		<xacro:module_macro name="module_02" parent_link="world" x="0.0" y="5.0" z="0.0" roll="0.0" pitch="0.0" yaw="1.5" />
-		<xacro:module_macro name="module_03" parent_link="world" x="-5.0" y="0.0" z="0.0" roll="0.0" pitch="0.0" yaw="3.0" />
-		<xacro:module_macro name="module_04" parent_link="world" x="0.0" y="-5.0" z="0.0" roll="0.0" pitch="0.0" yaw="-1.5" />
-		<xacro:module_macro name="module_05" parent_link="world" x="2.0" y="-5.0" z="0.0" roll="0.0" pitch="0.0" yaw="-0.75" />
+		<xacro:module_macro name="module_01" start_id="0" parent_link="world" x="4.0" y="0.0" z="0.0" roll="0.0" pitch="0.0" yaw="0.0" />
+		<xacro:module_macro name="module_02" start_id="30" parent_link="world" x="0.0" y="3.0" z="0.0" roll="0.0" pitch="0.0" yaw="90" />
+		<xacro:module_macro name="module_03" start_id="60" parent_link="world" x="-3.0" y="0.0" z="0.0" roll="0.0" pitch="0.0" yaw="180" />
+		<xacro:module_macro name="module_04" start_id="90" parent_link="world" x="0.0" y="-3.0" z="0.0" roll="0.0" pitch="0.0" yaw="-90" />
+		<xacro:module_macro name="module_05" start_id="120" parent_link="world" x="2.5" y="2.5" z="0.0" roll="0.0" pitch="0.0" yaw="45" />
+		<xacro:module_macro name="module_06" start_id="150" parent_link="world" x="-2.5" y="2.5" z="0.0" roll="0.0" pitch="0.0" yaw="135" />
+		<xacro:module_macro name="module_07" start_id="180" parent_link="world" x="-2.5" y="-2.5" z="0.0" roll="0.0" pitch="0.0" yaw="225" />
+		<xacro:module_macro name="module_08" start_id="210" parent_link="world" x="2.5" y="-2.5" z="0.0" roll="0.0" pitch="0.0" yaw="-45" />
 	</world>
 </sdf>

File: ros2_ws/src/simulation/worlds/module.xacro (robot description, xacro)
@@ -2,13 +2,14 @@
 <robot xmlns:xacro="http://www.ros.org/wiki/xacro">
     <xacro:include filename="utils.xacro" />
-    <xacro:macro name="module_macro" params="name parent_link x y z roll pitch yaw">
+    <xacro:macro name="module_macro" params="name start_id parent_link x y z roll pitch yaw">
         <model name="${name}">
             <static>true</static>
+            <pose>${x} ${y} ${z} ${roll * pi / 180.0} ${pitch * pi / 180.0} ${yaw * pi / 180.0}</pose>
             <link name="${name}_link">
                 <visual name="${name}_visual">
-                    <pose>${x} ${y} ${z} ${roll} ${pitch} ${yaw}</pose>
+                    <pose>0.0 0.0 1.0 0.0 0.0 0.0</pose>
                     <geometry>
                         <box>
-                            <size>0.1 1.0 3.0</size>
+                            <size>0.02 1.5 2.0</size>
                         </box>
                     </geometry>
@@ -17,4 +18,39 @@
             </link>
         </model>
+        <model name="${name}_marker_${start_id}">
+            <static>true</static>
+            <pose>${x} ${y} ${z} ${roll * pi / 180.0} ${pitch * pi / 180.0} ${yaw * pi / 180.0}</pose>
+            <xacro:marker_macro name="marker" id="${start_id}" parent_link="${name}_link"
+                x="-0.011" y="0.0" z="1.0" roll="0.0" pitch="90.0" yaw="0.0"
+            />
+        </model>
+        <model name="${name}_marker_${start_id + 1}">
+            <static>true</static>
+            <pose>${x} ${y} ${z} ${roll * pi / 180.0} ${pitch * pi / 180.0} ${yaw * pi / 180.0}</pose>
+            <xacro:marker_macro name="marker" id="${start_id + 1}" parent_link="${name}_link"
+                x="-0.011" y="0.5" z="1.0" roll="0.0" pitch="90.0" yaw="0.0"
+            />
+        </model>
+        <model name="${name}_marker_${start_id + 2}">
+            <static>true</static>
+            <pose>${x} ${y} ${z} ${roll * pi / 180.0} ${pitch * pi / 180.0} ${yaw * pi / 180.0}</pose>
+            <xacro:marker_macro name="marker" id="${start_id + 2}" parent_link="${name}_link"
+                x="-0.011" y="-0.5" z="1.0" roll="0.0" pitch="90.0" yaw="0.0"
+            />
+        </model>
+        <model name="${name}_marker_${start_id + 3}">
+            <static>true</static>
+            <pose>${x} ${y} ${z} ${roll * pi / 180.0} ${pitch * pi / 180.0} ${yaw * pi / 180.0}</pose>
+            <xacro:marker_macro name="marker" id="${start_id + 3}" parent_link="${name}_link"
+                x="-0.011" y="0.0" z="1.5" roll="0.0" pitch="90.0" yaw="0.0"
+            />
+        </model>
+        <model name="${name}_marker_${start_id + 4}">
+            <static>true</static>
+            <pose>${x} ${y} ${z} ${roll * pi / 180.0} ${pitch * pi / 180.0} ${yaw * pi / 180.0}</pose>
+            <xacro:marker_macro name="marker" id="${start_id + 4}" parent_link="${name}_link"
+                x="-0.011" y="0.0" z="0.5" roll="0.0" pitch="90.0" yaw="0.0"
+            />
+        </model>
     </xacro:macro>
 </robot>

File: ros2_ws/src/simulation/worlds/utils.xacro (robot description, xacro)
@@ -9,3 +9,22 @@
         </material>
     </xacro:macro>
+    <xacro:macro name="marker_macro" params="parent_link name id x y z roll pitch yaw">
+        <model name="${name}_${id}">
+            <static>true</static>
+            <pose>${x} ${y} ${z} ${roll * pi / 180.0} ${pitch * pi / 180.0} ${yaw * pi / 180.0}</pose>
+            <link name="${name}_${id}_link">
+                <visual name="${name}_${id}_visual">
+                    <geometry>
+                        <cylinder>
+                            <radius>0.1</radius>
+                            <length>0.001</length>
+                        </cylinder>
+                    </geometry>
+                </visual>
+            </link>
+            <plugin filename="gz-sim-label-system" name="gz::sim::systems::Label">
+                <label>${id}</label>
+            </plugin>
+        </model>
+    </xacro:macro>
 </robot>
