Commit message: huge changes to record pcd and bmp. Implementation on TreeNode and SE3 structure and python generator script for groundtruth world

File: ros2_ws/src/simulation/worlds/empty.urdf.xacro (robot description, xacro)
@@ -1,4 +1,5 @@
 <?xml version="1.0"?>
-<sdf version="1.6">
+<sdf version="1.6" xmlns:xacro="http://www.ros.org/wiki/xacro">
+	<xacro:include filename="utils.xacro" />
 	<world name="empty_world">
 		<physics name="1ms" type="ignored">
@@ -13,5 +14,4 @@
 			filename="gz-sim-sensors-system"
 			name="gz::sim::systems::Sensors">
-			<render_engine>ogre2</render_engine>
 		</plugin>
 		<plugin
@@ -124,74 +124,5 @@
 			</link>
 		</model>
-		<model name="box">
-			<pose>0 0 0.5 0 0 0</pose>
-			<link name="box_link">
-				<inertial>
-					<inertia>
-						<ixx>1</ixx>
-						<ixy>0</ixy>
-						<ixz>0</ixz>
-						<iyy>1</iyy>
-						<iyz>0</iyz>
-						<izz>1</izz>
-					</inertia>
-					<mass>1.0</mass>
-				</inertial>
-				<collision name="box_collision">
-					<geometry>
-						<box>
-							<size>1 1 1</size>
-						</box>
-					</geometry>
-				</collision>
-				<visual name="box_visual">
-					<geometry>
-						<box>
-							<size>1 1 1</size>
-						</box>
-					</geometry>
-					<material>
-						<ambient>1 0 0 1</ambient>
-						<diffuse>1 0 0 1</diffuse>
-						<specular>1 0 0 1</specular>
-					</material>
-				</visual>
-			</link>
-		</model>
-		<model name="box2">
-			<pose>0 2 0.5 0 0 0</pose>
-			<link name="box_link">
-				<inertial>
-					<inertia>
-						<ixx>1</ixx>
-						<ixy>0</ixy>
-						<ixz>0</ixz>
-						<iyy>1</iyy>
-						<iyz>0</iyz>
-						<izz>1</izz>
-					</inertia>
-					<mass>1.0</mass>
-				</inertial>
-				<collision name="box_collision">
-					<geometry>
-						<box>
-							<size>1 1 1</size>
-						</box>
-					</geometry>
-				</collision>
-				<visual name="box_visual">
-					<geometry>
-						<box>
-							<size>1 1 1</size>
-						</box>
-					</geometry>
-					<material>
-						<ambient>1 0 0 1</ambient>
-						<diffuse>1 0 0 1</diffuse>
-						<specular>1 0 0 1</specular>
-					</material>
-				</visual>
-			</link>
-		</model>
+		<!-- OBJECTS -->
 	</world>
 </sdf>
